File: Hardware/schematic/VC5.kicad_pcb (KiCad board)
At the start: 2 copper layers, 230 x 70 mm, 84 parts, among them J2 Debug_output, Q1 BC337, U1 1.3in SH1106 OLED, U2 1.3in SH1106 OLED, U3 1.3in SH1106 OLED, U4 1.3in SH1106 OLED, U5 1.3in SH1106 OLED, U6 MCP23017

Commit message: adjustments to the PCB layout after schematic change
Parts:
- added ?: , , F.Cu at (168.9, 101.8)
Connections:
- A1 pad 24: /displays/CS1 -> /displays/CLK
- A1 pad 25: /displays/CLK -> /displays/DIN
- A1 pad 26: /displays/DIN -> /displays/CS1
Routing:
- net /displays/DIN: track 261.4 -> 285.2 mm, vias 1 -> 3
- net /displays/CS1: track 15.5 -> 10.4 mm
- net /displays/CLK: track 278.7 -> 281.2 mm, vias 1 -> 2
Changed lines of the file:
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@@
 		)
 	)
+	(footprint ""
+		(layer "F.Cu")
+		(at 168.91 101.76)
+		(property "Reference" ""
+			(at 0 0 0)
+			(layer "F.SilkS")
+			(effects
+				(font
+					(size 1.27 1.27)
+					(thickness 0.15)
+				)
+			)
+		)
+		(property "Value" ""
+			(at 0 0 0)
+			(layer "F.Fab")
+			(effects
+				(font
+					(size 1.27 1.27)
+					(thickness 0.15)
+				)
+			)
+		)
+		(property "Datasheet" ""
+			(at 0 0 0)
+			(layer "F.Fab")
+			(hide yes)
+			(effects
+				(font
+					(size 1.27 1.27)
+					(thickness 0.15)
+				)
+			)
+		)
+		(property "Description" ""
+			(at 0 0 0)
+			(layer "F.Fab")
+			(hide yes)
+			(effects
+				(font
+					(size 1.27 1.27)
+					(thickness 0.15)
+				)
+			)
+		)
+		(pad "1" thru_hole oval
+			(at 0 0 270)
+			(size 1.7 1.7)
+			(drill 1)
+			(layers "*.Cu" "*.Mask")
+			(remove_unused_layers no)
+			(net 1 "GND")
+			(pinfunction "GND")
+			(pintype "power_in")
+		)
+		(embedded_fonts no)
+	)
 	(footprint "Capacitor_THT:C_Disc_D5.0mm_W2.5mm_P2.50mm"
 		(layer "B.Cu")
@@
 			(layers "*.Cu" "*.Mask")
 			(remove_unused_layers no)
-			(net 10 "/displays/CS1")
+			(net 17 "/displays/CLK")
 			(pinfunction "GPIO18")
 			(pintype "bidirectional")
@@
 			(layers "*.Cu" "*.Mask")
 			(remove_unused_layers no)
-			(net 17 "/displays/CLK")
+			(net 6 "/displays/DIN")
 			(pinfunction "GPIO19")
 			(pintype "bidirectional")
@@
 			(layers "*.Cu" "*.Mask")
 			(remove_unused_layers no)
-			(net 6 "/displays/DIN")
+			(net 10 "/displays/CS1")
 			(pinfunction "GPIO20")
 			(pintype "bidirectional")
@@
 	)
 	(gr_text "GND"
+		(at 171.61 101.76 0)
+		(layer "F.SilkS")
+		(effects
+			(font
+				(size 1 1)
+				(thickness 0.15)
+			)
+		)
+	)
+	(gr_text "GND"
 		(at 80.69 69.8 0)
 		(layer "F.SilkS")
@@
 	)
 	(gr_text "GND"
+		(at 171.61 101.76 0)
+		(layer "B.SilkS")
+		(effects
+			(font
+				(size 1 1)
+				(thickness 0.15)
+			)
+			(justify mirror)
+		)
+	)
+	(gr_text "GND"
 		(at 174.89 74.95 0)
 		(layer "B.SilkS")
@@
 	)
 	(segment
-		(start 114.91 65.1)
-		(end 110.33 69.68)
+		(start 141.8 72.19)
+		(end 141.8 71.92)
 		(width 0.6)
 		(layer "F.Cu")
@@
 	)
 	(segment
+		(start 138.84 68.96)
+		(end 129.88 68.96)
+		(width 0.6)
+		(layer "F.Cu")
+		(net 6)
+	)
+	(segment
 		(start 145.529 79.981)
 		(end 143.28 79.981)
@@
 	)
 	(segment
+		(start 141.8 76.32)
+		(end 141.8 72.19)
+		(width 0.6)
+		(layer "F.Cu")
+		(net 6)
+	)
+	(segment
 		(start 160.41 65.1)
 		(end 145.529 79.981)
@@
 	)
 	(segment
+		(start 118.77 68.96)
+		(end 114.91 65.1)
+		(width 0.6)
+		(layer "F.Cu")
+		(net 6)
+	)
+	(segment
 		(start 138.141 79.981)
 		(end 138.14 79.98)
@@
 	)
 	(segment
-		(start 104.5 69.68)
-		(end 102.25 71.93)
+		(start 191.029 79.981)
+		(end 242.719 79.981)
 		(width 0.6)
 		(layer "F.Cu")
@@
 	)
 	(segment
-		(start 191.029 79.981)
-		(end 242.719 79.981)
+		(start 138.94 69.06)
+		(end 138.84 68.96)
 		(width 0.6)
 		(layer "F.Cu")
@@
 	)
 	(segment
-		(start 110.33 69.68)
-		(end 104.5 69.68)
+		(start 138.14 79.98)
+		(end 141.8 76.32)
 		(width 0.6)
 		(layer "F.Cu")
@@
 	)
 	(segment
+		(start 141.8 71.92)
+		(end 138.94 69.06)
+		(width 0.6)
+		(layer "F.Cu")
+		(net 6)
+	)
+	(segment
 		(start 205.91 65.1)
 		(end 191.029 79.981)
@@
 		(net 6)
 	)
+	(via
+		(at 118.77 68.96)
+		(size 0.8)
+		(drill 0.3)
+		(layers "F.Cu" "B.Cu")
+		(net 6)
+	)
+	(via
+		(at 129.88 68.96)
+		(size 0.8)
+		(drill 0.3)
+		(layers "F.Cu" "B.Cu")
+		(net 6)
+	)
 	(segment
-		(start 97.87 76.31)
-		(end 102.25 71.93)
+		(start 95.33 76.31)
+		(end 99.71 71.93)
 		(width 0.6)
 		(layer "B.Cu")
@@
 	)
 	(segment
+		(start 107.76 79.98)
+		(end 99.71 71.93)
+		(width 0.6)
+		(layer "B.Cu")
+		(net 6)
+	)
+	(segment
+		(start 129.88 68.96)
+		(end 118.77 68.96)
+		(width 0.6)
+		(layer "B.Cu")
+		(net 6)
+	)
+	(segment
 		(start 83.295572 76.31)
-		(end 97.87 76.31)
+		(end 92.58 76.31)
 		(width 0.6)
 		(layer "B.Cu")
@@
 	)
 	(segment
-		(start 138.14 79.98)
-		(end 110.3 79.98)
+		(start 92.58 76.31)
+		(end 95.33 76.31)
 		(width 0.6)
 		(layer "B.Cu")
@@
 	)
 	(segment
-		(start 110.3 79.98)
-		(end 102.25 71.93)
+		(start 138.14 79.98)
+		(end 107.76 79.98)
 		(width 0.6)
 		(layer "B.Cu")
@@
 	)
 	(segment
-		(start 106.86 68.07)
-		(end 101.03 68.07)
+		(start 107.86 67.07)
+		(end 107.11 67.07)
 		(width 0.6)
 		(layer "F.Cu")
@@
 	)
 	(segment
-		(start 101.03 68.07)
-		(end 97.17 71.93)
+		(start 109.83 65.1)
+		(end 107.86 67.07)
 		(width 0.6)
 		(layer "F.Cu")
@@
 	)
 	(segment
-		(start 109.83 65.1)
-		(end 106.86 68.07)
+		(start 107.11 67.07)
+		(end 102.25 71.93)
 		(width 0.6)
 		(layer "F.Cu")
@@
 	)
 	(segment
-		(start 94.29 77.35)
-		(end 99.71 71.93)
+		(start 97.17 71.93)
+		(end 97.17 76.1)
 		(width 0.6)
 		(layer "F.Cu")
@@
 	)
 	(segment
-		(start 108.59 68.88)
+		(start 108.82 68.65)
 		(end 112.37 65.1)
 		(width 0.6)
@@
 	)
 	(segment
-		(start 99.71 71.93)
-		(end 102.76 68.88)
+		(start 97.17 76.1)
+		(end 97.19 76.12)
 		(width 0.6)
 		(layer "F.Cu")
@@
 	)
 	(segment
-		(start 102.76 68.88)
-		(end 108.59 68.88)
+		(start 107.639336 68.65)
+		(end 108.82 68.65)
 		(width 0.6)
 		(layer "F.Cu")
@@
 	)
 	(via
-		(at 94.29 77.35)
-		(size 0.6)
+		(at 107.639336 68.65)
+		(size 0.8)
 		(drill 0.3)
 		(layers "F.Cu" "B.Cu")
 		(net 17)
 	)
-	(segment
-		(start 184.4 82.97)
-		(end 161.11 82.97)
-		(width 0.6)
-		(layer "B.Cu")
+	(via
+		(at 97.19 76.12)
+		(size 0.8)
+		(drill 0.3)
+		(layers "F.Cu" "B.Cu")
 		(net 17)
 	)
 	(segment
-		(start 77.121786 71.269)
-		(end 73.039 71.269)
+		(start 184.4 82.97)
+		(end 161.11 82.97)
 		(width 0.6)
 		(layer "B.Cu")
@@
 	)
 	(segment
+		(start 100.11 68.99)
+		(end 97.17 71.93)
+		(width 0.6)
+		(layer "B.Cu")
+		(net 17)
+	)
+	(segment
+		(start 91.72 77.35)
+		(end 83.202786 77.35)
+		(width 0.6)
+		(layer "B.Cu")
+		(net 17)
+	)
+	(segment
+		(start 95.96 77.35)
+		(end 94.29 77.35)
+		(width 0.6)
+		(layer "B.Cu")
+		(net 17)
+	)
+	(segment
+		(start 100.45 68.65)
+		(end 107.639336 68.65)
+		(width 0.6)
+		(layer "B.Cu")
+		(net 17)
+	)
+	(segment
 		(start 203.37 65.1)
 		(end 185.5 82.97)
@@
 	)
 	(segment
-		(start 73.039 71.269)
-		(end 66.87 65.1)
+		(start 97.19 76.12)
+		(end 95.96 77.35)
+		(width 0.6)
+		(layer "B.Cu")
+		(net 17)
+	)
+	(segment
+		(start 77.121786 71.269)
+		(end 73.039 71.269)
 		(width 0.6)
 		(layer "B.Cu")
@@
 	)
 	(segment
-		(start 94.29 77.35)
-		(end 83.202786 77.35)
+		(start 100.11 68.99)
+		(end 100.45 68.65)
 		(width 0.6)
 		(layer "B.Cu")
@@
 	)
 	(segment
+		(start 73.039 71.269)
+		(end 66.87 65.1)
+		(width 0.6)
+		(layer "B.Cu")
+		(net 17)
+	)
+	(segment
 		(start 185.5 82.97)
 		(end 184.4 82.97)
 		(width 0.6)
 		(layer "B.Cu")
+		(net 17)
+	)
+	(segment
+		(start 94.29 77.35)
+		(end 91.72 77.35)
+		(width 0.6)
+		(layer "B.Cu")
